File: Driver_Board.kicad_pcb (KiCad board)
At the start: 2 copper layers, 112.5 x 71.6 mm, 26 parts, among them J1 200, J2 100, J3 10, J4 Conn_01x04, J5 Conn_01x04, J6 Control

Commit message: Основа ADUM4135
Parts:
- removed H1, H2, H3: MountingHole, MountingHole:MountingHole_3.2mm_M3
- removed J2: 100, Connector_PinSocket_2.54mm:PinSocket_2x05_P2.54mm_Vertical
- removed J3: 10, Connector_PinSocket_2.54mm:PinSocket_2x05_P2.54mm_Vertical
- removed J4, J5: Conn_01x04, IGBT_Modul:IGBT_Control
- removed J6: Control, Connector_IDC:IDC-Header_2x04_P2.54mm_Vertical
- added C6: 10u, Capacitor_SMD:C_1210_3225Metric_Pad1.33x2.70mm_HandSolder, F.Cu at (77.0, 62.7)
- added C7: 56p, Capacitor_SMD:C_0805_2012Metric_Pad1.18x1.45mm_HandSolder, F.Cu at (79.5, 78.7)
- added D3: BZT52C10-7-F, Diode_SMD:D_SOD-123, F.Cu at (99.6, 85.1)
- added D4: BZT52C10-7-F, Diode_SMD:D_SOD-123, F.Cu at (104.1, 89.9)
- added D5: MURS360T3G, Diode_SMD:D_SMA_Handsoldering, F.Cu at (116.1, 87.2)
- added D6: MURS360T3G, Diode_SMD:D_SMA_Handsoldering, F.Cu at (120.1, 87.1)
- added D7: LED_Small, LED_SMD:LED_0805_2012Metric_Pad1.15x1.40mm_HandSolder, F.Cu at (77.2, 87.4)
- added D8: LED_Small, LED_SMD:LED_0805_2012Metric_Pad1.15x1.40mm_HandSolder, F.Cu at (77.2, 83.1)
- added R12: 10k, Resistor_SMD:R_0805_2012Metric_Pad1.20x1.40mm_HandSolder, F.Cu at (81.8, 83.1)
- added R13: 380, Resistor_SMD:R_0805_2012Metric_Pad1.20x1.40mm_HandSolder, F.Cu at (79.5, 87.4)
- added R14: 500, Resistor_SMD:R_0805_2012Metric_Pad1.20x1.40mm_HandSolder, F.Cu at (79.5, 83.1)
- added R15: 2.2k, Resistor_SMD:R_0805_2012Metric_Pad1.20x1.40mm_HandSolder, F.Cu at (99.6, 80.2)
- added R9: 3.9, Resistor_SMD:R_1206_3216Metric_Pad1.30x1.75mm_HandSolder, F.Cu at (105.4, 77.0)
- added U1: TEC2-1213WI, Converter_DCDC:Converter_DCDC_TRACO_TMR-xxxx_THT, F.Cu at (81.4, 61.1)
- C1, C2: value C_Small -> 0.1u; moved to F.Cu
- C3: value CCFG -> 220p; moved to F.Cu
- C4: value 1n -> 0.1u; moved to F.Cu
- C5: value 100n -> 0.1u
- D1: value D_Small -> ADUM4135; footprint Diode_SMD:D_SMA_Handsoldering -> Package_SO:SOIC-16W_7.5x10.3mm_P1.27mm
- D2: value D_Small -> MURS360T3G
- J1: value 200 -> Conn_02x07_Odd_Even; footprint Connector_PinSocket_2.54mm:PinSocket_2x05_P2.54mm_Vertical -> Connector_IDC:IDC-Header_2x07-1MP_P2.54mm_Latch_Vertical
- R1: value 30.1k -> 120; footprint Resistor_SMD:R_2512_6332Metric_Pad1.40x3.35mm_HandSolder -> Resistor_SMD:R_0805_2012Metric_Pad1.20x1.40mm_HandSolder; moved to F.Cu
- R10: value 10k -> 12k; footprint Resistor_SMD:R_2512_6332Metric_Pad1.40x3.35mm_HandSolder -> Resistor_SMD:R_1206_3216Metric_Pad1.30x1.75mm_HandSolder; moved to F.Cu
- R11: value 0 -> 12k; footprint Resistor_SMD:R_2512_6332Metric_Pad1.40x3.35mm_HandSolder -> Resistor_SMD:R_1206_3216Metric_Pad1.30x1.75mm_HandSolder; moved to F.Cu
- R2: value RON -> 120; footprint Resistor_SMD:R_2512_6332Metric_Pad1.40x3.35mm_HandSolder -> Resistor_SMD:R_0805_2012Metric_Pad1.20x1.40mm_HandSolder
- R3: value 50 -> 12k; footprint Resistor_SMD:R_2512_6332Metric_Pad1.40x3.35mm_HandSolder -> Resistor_SMD:R_1206_3216Metric_Pad1.30x1.75mm_HandSolder
- R4: value 511 -> 3.9; footprint Resistor_SMD:R_2512_6332Metric_Pad1.40x3.35mm_HandSolder -> Resistor_SMD:R_1206_3216Metric_Pad1.30x1.75mm_HandSolder
- R5: value ROFF -> 3.9; footprint Resistor_SMD:R_2512_6332Metric_Pad1.40x3.35mm_HandSolder -> Resistor_SMD:R_1206_3216Metric_Pad1.30x1.75mm_HandSolder
- R6: value R1 -> 3.9; footprint Resistor_SMD:R_2512_6332Metric_Pad1.40x3.35mm_HandSolder -> Resistor_SMD:R_1206_3216Metric_Pad1.30x1.75mm_HandSolder; moved to F.Cu
- R7: value 10k -> 3.9; footprint Resistor_SMD:R_2512_6332Metric_Pad1.40x3.35mm_HandSolder -> Resistor_SMD:R_1206_3216Metric_Pad1.30x1.75mm_HandSolder; moved to F.Cu
- R8: value 30.1k -> 3.9; footprint Resistor_SMD:R_2512_6332Metric_Pad1.40x3.35mm_HandSolder -> Resistor_SMD:R_1206_3216Metric_Pad1.30x1.75mm_HandSolder
- moved J1 89.1 mm to (63.5, 84.1), turned to 180 degrees
- moved C5 88.7 mm to (74.9, 83.1), turned to -90 degrees
- moved R1 71.9 mm to (77.2, 78.7), turned to 90 degrees
- moved R2 71.4 mm to (81.8, 87.4)
- moved C1 70.9 mm to (81.8, 78.7), turned to 90 degrees
- moved C4 70.0 mm to (74.9, 87.4)
- moved C2 68.2 mm to (97.8, 69.1), turned to 180 degrees
- moved R8 66.7 mm to (108.0, 77.0), turned to 90 degrees
- moved R7 66.7 mm to (102.9, 71.4), turned to -90 degrees
- moved R5 59.3 mm to (102.9, 77.0)
- moved R10 57.0 mm to (102.6, 85.1), turned to -90 degrees
- moved C3 55.7 mm to (96.8, 85.1), turned to -90 degrees
- moved R3 52.3 mm to (105.4, 85.1)
- moved D1 48.5 mm to (89.4, 74.2), turned to 0 degrees
- moved R6 43.0 mm to (108.0, 71.4), turned to -90 degrees
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Connections:
- C1 pad 1: GNDPWR -> GNDA
- C1 pad 2: /CFG -> +5VD
- C2 pad 1: GNDPWR -> +15V
- C2 pad 2: Net-(C2-Pad2) -> E_IGBT
- C3 pad 1: /CFG -> Desat
- C3 pad 2: GNDPWR -> E_IGBT
- C4 pad 1: GND -> RDY
- C4 pad 2: /BOT_IN -> GNDA
- C5 pad 1: GND -> FLT
- C5 pad 2: /ERR_OUT -> GNDA
- D1 pad 1: Net-(D1-Pad1) -> GNDA
- D1 pad 2: Net-(D1-Pad2) -> IN+
- D2 pad 1: /E1 -> Net-(D2-Pad1)
- D2 pad 2: Net-(D1-Pad1) -> Net-(D2-Pad2)
- J1 pad 1: /CFG -> RDY
- J1 pad 10: Net-(C2-Pad2) -> GNDA
- J1 pad 2: Net-(J1-Pad2) -> GNDA
- J1 pad 3: /SEC_BOT -> FLT
- J1 pad 4: /SEC_BOT -> GNDA
- J1 pad 5: Net-(J1-Pad5) -> RST
- J1 pad 6: Net-(R5-Pad1) -> GNDA
- J1 pad 7: GNDPWR -> IN-
- J1 pad 8: GNDPWR -> GNDA
- J1 pad 9: Net-(J1-Pad9) -> IN+
- R1 pad 1: /CFG -> RST
- R1 pad 2: /SEC_BOT -> Net-(C7-Pad2)
- R10 pad 1: GNDPWR -> Desat
- R10 pad 2: /GATE -> Net-(D4-Pad1)
- R11 pad 1: Net-(J2-Pad2) -> Desat
- R11 pad 2: /E1 -> Net-(D4-Pad1)
- R2 pad 1: /GATE -> +5VD
- R2 pad 2: Net-(J1-Pad5) -> RDY
- R3 pad 1: /GATE -> Desat
- R3 pad 2: Net-(J1-Pad9) -> Net-(D4-Pad1)
- R4 pad 1: Net-(J1-Pad2) -> Net-(D1-Pad14)
- R4 pad 2: Net-(D1-Pad2) -> G_IGBT
- R5 pad 1: Net-(R5-Pad1) -> Net-(D1-Pad12)
- R5 pad 2: /GATE -> G_IGBT
- R6 pad 1: GNDPWR -> Net-(D1-Pad14)
- R6 pad 2: /CFG -> G_IGBT
- R7 pad 1: GND -> Net-(D1-Pad14)
- R7 pad 2: /BOT_IN -> G_IGBT
- R8 pad 1: /ERR_OUT -> Net-(D1-Pad12)
- R8 pad 2: +15V -> G_IGBT
Routing:
- net /BOT_IN: track 57.5 -> 0.00 mm
- net /ERR_OUT: track 52.8 -> 0.00 mm
- net RDY: track 0.00 -> 43.8 mm, vias 0 -> 2
- net FLT: track 0.00 -> 30.2 mm, vias 0 -> 3
- net /E1: track 27.7 -> 0.00 mm
- net GND: track 26.0 -> 0.00 mm
- net Desat: track 0.00 -> 23.9 mm
- net IN-: track 0.00 -> 23.0 mm
- net IN+: track 0.00 -> 22.5 mm
- net Net-(R5-Pad1): track 21.0 -> 0.00 mm
- net E_IGBT: track 0.00 -> 18.2 mm, vias 0 -> 3
- net GNDA: track 0.00 -> 17.5 mm, vias 0 -> 5
- net Net-(J1-Pad2): track 16.5 -> 0.00 mm
- net Net-(D1-Pad12): track 0.00 -> 16.2 mm
- net Net-(D1-Pad14): track 0.00 -> 15.1 mm
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- added copper zone on In1.Cu, net +15V
- added copper zone on In1.Cu, net +5VD
- added copper zone on In2.Cu, net E_IGBT
- added copper zone on In2.Cu, net GNDA
- added copper zone on F.Cu, net G_IGBT
- added copper zone on In1.Cu, net VAA
- removed copper zone on F.Cu, net +15V
- removed copper zone on B.Cu, net /CFG
- removed copper zone on F.Cu, net /GATE
- removed copper zone on F.Cu, net GND
- removed copper zone on B.Cu, net GNDPWR
Other:
- board size 112.5 x 71.6 mm -> 66.5 x 44.4 mm
- copper layers 2 -> 4

Commit message: Плата на два модуля
Parts:
- removed D2, D5: MURS360T3G, Diode_SMD:D_SMA_Handsoldering
- removed R11: 12k, Resistor_SMD:R_1206_3216Metric_Pad1.30x1.75mm_HandSolder
- added J2: IGBT, IGBT_Modul:IGBT_Gate, F.Cu at (46.0, 49.5)
- added J3: IGBT_Diode, IGBT_Modul:IGBT_Gate, F.Cu at (119.1, 49.5)
- added J4: Conn_01x01, Connector Power:Wire, F.Cu at (132.1, 78.2)
- C2: moved to B.Cu
- R10: value 12k -> 100; footprint Resistor_SMD:R_1206_3216Metric_Pad1.30x1.75mm_HandSolder -> Resistor_SMD:R_0805_2012Metric_Pad1.20x1.40mm_HandSolder
- R3: value 12k -> 1.6k
- moved J1 39.9 mm to (23.6, 84.1)
- moved R5 34.0 mm to (130.8, 57.7)
- moved R9 34.0 mm to (133.3, 57.7)
- moved R8 34.0 mm to (135.9, 57.7)
- moved R7 28.4 mm to (127.8, 57.7), turned to 90 degrees
- moved R10 26.5 mm to (79.8, 71.6)
- moved R4 24.1 mm to (125.2, 57.7), turned to 90 degrees
- moved R6 20.1 mm to (122.7, 57.7), turned to 90 degrees
- moved D4 11.6 mm to (114.3, 84.3)
- moved R15 7.75 mm to (94.5, 86.1), turned to -90 degrees
- moved D6 3.95 mm to (122.9, 84.3), turned to 180 degrees
- moved R3 3.14 mm to (108.5, 84.3), turned to 0 degrees
- moved C2 2.55 mm to (98.0, 71.6), turned to 90 degrees
- moved C3 1.29 mm to (97.5, 86.1)
- moved D3 1.29 mm to (100.3, 86.1)
Connections:
- D4 pad 2: Net-(D2-Pad2) -> Net-(D4-Pad2)
- D6 pad 1: K_IGBT -> C_IGBT
- D6 pad 2: Net-(D5-Pad1) -> Net-(D4-Pad2)
- R10 pad 1: Desat -> IN+
- R10 pad 2: Net-(D4-Pad1) -> IN-
Routing:
- net Net-(D1-Pad12): track 16.2 -> 56.0 mm
- net Net-(D1-Pad14): track 15.1 -> 46.8 mm
- net G_IGBT: track 10.1 -> 40.6 mm, vias 2 -> 0
- net RDY: track 43.8 -> 51.0 mm
- net Desat: track 23.9 -> 30.9 mm
- net +15V: track 2.33 -> 9.29 mm
- net C_IGBT: track 0.00 -> 6.64 mm
- net Net-(D4-Pad1): track 9.09 -> 2.64 mm
- net Net-(D2-Pad2): track 6.35 -> 0.00 mm
- net FLT: track 30.2 -> 36.3 mm
- net Net-(D4-Pad2): track 0.00 -> 4.49 mm
- net Net-(D2-Pad1): track 4.08 -> 0.00 mm
- net Net-(D5-Pad1): track 4.08 -> 0.00 mm
- net E_IGBT: track 18.2 -> 16.1 mm, vias 3 -> 5
- added copper zone on F.Cu, net E_IGBT
Other:
- board outline removed

Commit message: Первая версия в производство
Parts:
- removed J2: IGBT, IGBT_Modul:IGBT_Gate
- added H1: MountingHole, MountingHole:MountingHole_3.2mm_M3, F.Cu at (120.7, 97.0)
- added H3: MountingHole, MountingHole:MountingHole_3.2mm_M3, F.Cu at (73.7, 97.0)
- moved J1 41.4 mm to (65.0, 85.6)
- moved J4 18.2 mm to (118.6, 65.9)
- moved R4 14.9 mm to (110.5, 59.9)
- moved R5 14.9 mm to (116.1, 59.9)
- moved R6 14.9 mm to (108.0, 59.9)
- moved R7 14.9 mm to (113.0, 59.9)
- moved R9 14.9 mm to (118.6, 59.9)
- moved R8 14.9 mm to (121.2, 59.9)
- moved J3 11.2 mm to (108.2, 52.1)
- moved D6 5.29 mm to (118.6, 81.3), turned to -90 degrees
- moved R3 3.30 mm to (105.2, 84.3)
- moved D4 2.54 mm to (111.8, 84.3)
Routing:
- net Net-(D1-Pad12): track 56.0 -> 34.1 mm
- net Net-(D1-Pad14): track 46.8 -> 28.1 mm
- net G_IGBT: track 40.6 -> 23.7 mm
- net Desat: track 30.9 -> 24.7 mm
- net RDY: track 51.0 -> 48.6 mm
- net RST: track 14.0 -> 12.5 mm
- net FLT: track 36.3 -> 35.0 mm
- net Net-(D4-Pad2): track 4.49 -> 5.43 mm
- net Net-(D4-Pad1): track 2.64 -> 3.40 mm
- net IN+: track 22.5 -> 21.9 mm
- added copper zone on B.Cu, net E_IGBT
- removed copper zone on F.Cu, net E_IGBT
Other:
- board outline added: 66.5 x 52.3 mm
- board text added: "C_IGBT"
- board text added: "E"
- board text added: "G"
