File: Driver_Board.kicad_sch (KiCad schematic)
At the start: 26 parts, among them J1 200, J2 100, J3 10, J4 Conn_01x04, J5 Conn_01x04, J6 Control

Commit message: Основа ADUM4135
Parts:
- removed D1: D_Small, Diode_SMD:D_SMA_Handsoldering, symbol Device:D_Small
- removed H1, H2, H3: MountingHole, MountingHole:MountingHole_3.2mm_M3, symbol Mechanical:MountingHole
- removed J1: 200, Connector_PinSocket_2.54mm:PinSocket_2x05_P2.54mm_Vertical, symbol Connector_Generic:Conn_02x05_Odd_Even
- removed J2: 100, Connector_PinSocket_2.54mm:PinSocket_2x05_P2.54mm_Vertical, symbol Connector_Generic:Conn_02x05_Odd_Even
- removed J3: 10, Connector_PinSocket_2.54mm:PinSocket_2x05_P2.54mm_Vertical, symbol Connector_Generic:Conn_02x05_Odd_Even
- removed J4, J5: Conn_01x04, IGBT_Modul:IGBT_Control, symbol Connector_Generic:Conn_01x04
- removed J6: Control, Connector_IDC:IDC-Header_2x04_P2.54mm_Vertical, symbol Connector_Generic:Conn_02x04_Odd_Even
- added C6: 10u, Capacitor_SMD:C_1210_3225Metric_Pad1.33x2.70mm_HandSolder, symbol Device:C_Small
- added C7: 56p, Capacitor_SMD:C_0805_2012Metric_Pad1.18x1.45mm_HandSolder, symbol Device:C_Small
- added D1: ADUM4135, Package_SO:SOIC-16W_7.5x10.3mm_P1.27mm, symbol ADUM_Driver:ADUM4135
- added D3, D4: BZT52C10-7-F, Diode_SMD:D_SOD-123, symbol Device:D_Zener_Small
- added D5, D6: MURS360T3G, Diode_SMD:D_SMA_Handsoldering, symbol Device:D_Small
- added D7, D8: LED_Small, LED_SMD:LED_0805_2012Metric_Pad1.15x1.40mm_HandSolder, symbol Device:LED_Small
- added J1: Conn_02x07_Odd_Even, Connector_IDC:IDC-Header_2x07-1MP_P2.54mm_Latch_Vertical, symbol Connector_Generic:Conn_02x07_Odd_Even
- added R12: 10k, Resistor_SMD:R_0805_2012Metric_Pad1.20x1.40mm_HandSolder, symbol Device:R_Small
- added R13: 380, Resistor_SMD:R_0805_2012Metric_Pad1.20x1.40mm_HandSolder, symbol Device:R_Small
- added R14: 500, Resistor_SMD:R_0805_2012Metric_Pad1.20x1.40mm_HandSolder, symbol Device:R_Small
- added R15: 2.2k, Resistor_SMD:R_0805_2012Metric_Pad1.20x1.40mm_HandSolder, symbol Device:R_Small
- added R9: 3.9, Resistor_SMD:R_1206_3216Metric_Pad1.30x1.75mm_HandSolder, symbol Device:R_Small
- added U1: TEC2-1213WI, Converter_DCDC:Converter_DCDC_TRACO_TMR-xxxx_THT, symbol Converter_DCDC:TEC2-1213WI
- C1, C2: value C_Small -> 0.1u
- C3: value CCFG -> 220p
- C4: value 1n -> 0.1u
- C5: value 100n -> 0.1u
- D2: value D_Small -> MURS360T3G
- R1: value 30.1k -> 120; footprint Resistor_SMD:R_2512_6332Metric_Pad1.40x3.35mm_HandSolder -> Resistor_SMD:R_0805_2012Metric_Pad1.20x1.40mm_HandSolder
- R10: value 10k -> 12k; footprint Resistor_SMD:R_2512_6332Metric_Pad1.40x3.35mm_HandSolder -> Resistor_SMD:R_1206_3216Metric_Pad1.30x1.75mm_HandSolder
- R11: value 0 -> 12k; footprint Resistor_SMD:R_2512_6332Metric_Pad1.40x3.35mm_HandSolder -> Resistor_SMD:R_1206_3216Metric_Pad1.30x1.75mm_HandSolder
- R2: value RON -> 120; footprint Resistor_SMD:R_2512_6332Metric_Pad1.40x3.35mm_HandSolder -> Resistor_SMD:R_0805_2012Metric_Pad1.20x1.40mm_HandSolder
- R3: value 50 -> 12k; footprint Resistor_SMD:R_2512_6332Metric_Pad1.40x3.35mm_HandSolder -> Resistor_SMD:R_1206_3216Metric_Pad1.30x1.75mm_HandSolder
- R4: value 511 -> 3.9; footprint Resistor_SMD:R_2512_6332Metric_Pad1.40x3.35mm_HandSolder -> Resistor_SMD:R_1206_3216Metric_Pad1.30x1.75mm_HandSolder
- R5: value ROFF -> 3.9; footprint Resistor_SMD:R_2512_6332Metric_Pad1.40x3.35mm_HandSolder -> Resistor_SMD:R_1206_3216Metric_Pad1.30x1.75mm_HandSolder
- R6: value R1 -> 3.9; footprint Resistor_SMD:R_2512_6332Metric_Pad1.40x3.35mm_HandSolder -> Resistor_SMD:R_1206_3216Metric_Pad1.30x1.75mm_HandSolder
- R7: value 10k -> 3.9; footprint Resistor_SMD:R_2512_6332Metric_Pad1.40x3.35mm_HandSolder -> Resistor_SMD:R_1206_3216Metric_Pad1.30x1.75mm_HandSolder
- R8: value 30.1k -> 3.9; footprint Resistor_SMD:R_2512_6332Metric_Pad1.40x3.35mm_HandSolder -> Resistor_SMD:R_1206_3216Metric_Pad1.30x1.75mm_HandSolder
Connections:
- net +15V: now also C2.1, D1.13 (Vdd2), R15.2, U1.6 (+VOUT); no longer R8.2
- net GND2: now reaches C2.2
- net GND2: now also C3.2, D1.11 (GND2), D1.16 (Vss2), D1.9 (Vss2), D3.2 (A), U1.7 (-VOUT)
- net at R4.1: now also R6.1, R7.1, D1.14 (Vout_on)
- net RDY: now reaches R2.2
- net RDY: now also C4.1, D1.4 (READY), J1.1 (Pin_1), R13.1
- net at R5.1: now also R8.1, D1.12 (Vout_off), R9.1
- net at R3.2: now also R10.2, R11.2, D4.1 (K)
- net G_IGBT: now reaches R4.2
- net G_IGBT: now also R5.2, R6.2, R7.2, R8.2, D1.15 (GATE_SENSE), R9.2
- net at D2.2 (A): now also D4.2 (A)
- net Desat: now reaches R11.1
- net Desat: now also C3.1, R10.1, R3.1, D1.10 (DESAT), D3.1 (K), R15.1
- net BOT_IN renamed GNDA
- net GNDA: now also C1.1, C5.2, C6.2, C7.1, D1.1 (Vss1), D1.8 (Vss1), D7.1 (K), J1.10 (Pin_10), J1.12 (Pin_12), J1.14 (Pin_14), J1.2 (Pin_2), J1.4 (Pin_4), J1.6 (Pin_6), J1.8 (Pin_8), U1.1 (-VIN); no longer R7.2
- removed net CFG: C1.2, C3.1, R1.1, R6.2
- net E1: no longer names the net of D2.1 (K)
- net E1: now also D5.2 (A); no longer R11.2
- removed net ERR_OUT: C5.2, R8.1
- removed net GATE: R10.2, R2.1, R3.1, R5.2
- removed net GND: C4.1, C5.1, R7.1
- removed net GNDPWR: C1.1, C2.1, C3.2, R10.1, R6.1
- net SEC_BOT: no longer names the net of R1.2
- net SEC_BOT: now also C7.2, D1.6 (~{RESET})
- new net: D5.1 (K), D6.2 (A)
- new net: D7.2 (A), R13.2
- new net: D8.2 (A), R14.2
- new net +5VD: C1.2, D1.7 (Vdd1), J1.11 (Pin_11), R12.1, R14.1, R2.1
- new net FLT: C5.1, D1.5 (~{FAULT}), D8.1 (K), J1.3 (Pin_3), R12.2
- new net IN+: D1.2 (Vi+), J1.9 (Pin_9)
- new net IN-: D1.3 (Vi-), J1.7 (Pin_7)
- new net K_IGBT: D6.1 (K)
- new net RST: J1.5 (Pin_5), R1.1
- new net VAA: C6.1, J1.13 (Pin_13), U1.2 (+VIN)
- no-connect marks 9 -> 1

Commit message: Плата на два модуля
Parts:
- removed D2, D5: MURS360T3G, Diode_SMD:D_SMA_Handsoldering, symbol Device:D_Small
- removed R11: 12k, Resistor_SMD:R_1206_3216Metric_Pad1.30x1.75mm_HandSolder, symbol Device:R_Small
- added J2: IGBT, IGBT_Modul:IGBT_Gate, symbol Connector_Generic:Conn_01x04
- added J3: IGBT_Diode, IGBT_Modul:IGBT_Gate, symbol Connector_Generic:Conn_01x04
- added J4: Conn_01x01, Connector Power:Wire, symbol Connector_Generic:Conn_01x01
- R10: value 12k -> 100; footprint Resistor_SMD:R_1206_3216Metric_Pad1.30x1.75mm_HandSolder -> Resistor_SMD:R_0805_2012Metric_Pad1.20x1.40mm_HandSolder
- R3: value 12k -> 1.6k
Connections:
- net Desat: no longer R10.1
- net GND2: now also J3.3 (Pin_3)
- net G_IGBT: now also J3.4 (Pin_4)
- net IN+: now also R10.1
- net IN-: now also R10.2
- net at D6.2 (A): now also D4.2 (A)
- net at D4.1 (K), R3.2: no longer R10.2
- net K_IGBT renamed C_IGBT
- net C_IGBT: now also J4.1 (Pin_1)
- new net: J2.1 (Pin_1), J2.2 (Pin_2)
- new net: J2.3 (Pin_3), J2.4 (Pin_4)
- no-connect marks 1 -> 3
Other:
- moved on the sheet: D6

Commit message: Первая версия в производство
Parts:
- removed J2: IGBT, IGBT_Modul:IGBT_Gate, symbol Connector_Generic:Conn_01x04
- added H1, H3: MountingHole, MountingHole:MountingHole_3.2mm_M3, symbol Mechanical:MountingHole
Changed lines of the file:
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@@
-    (stroke (width 0) (type default) (color 0 0 0 0))
-  )
-  (wire (pts (xy 254.508 72.898) (xy 254.508 75.438))
     (stroke (width 0) (type default) (color 0 0 0 0))
   )
@@
   )
   (wire (pts (xy 72.644 85.598) (xy 73.66 85.598))
-    (stroke (width 0) (type default) (color 0 0 0 0))
-  )
-  (wire (pts (xy 254.508 67.818) (xy 254.508 70.358))
     (stroke (width 0) (type default) (color 0 0 0 0))
   )
@@
     (pin "2")
   )
-  (symbol (lib_id "Connector_Generic:Conn_01x04") (at 259.588 70.358 0) (unit 1)
-    (in_bom yes) (on_board yes) (fields_autoplaced)
-    (property "Reference" "J2" (id 0) (at 261.62 70.3579 0)
-      (effects (font (size 1.27 1.27)) (justify left))
-    )
-    (property "Value" "IGBT" (id 1) (at 261.62 72.8979 0)
-      (effects (font (size 1.27 1.27)) (justify left))
-    )
-    (property "Footprint" "IGBT_Modul:IGBT_Gate" (id 2) (at 259.588 70.358 0)
-      (effects (font (size 1.27 1.27)) hide)
-    )
-    (property "Datasheet" "~" (id 3) (at 259.588 70.358 0)
-      (effects (font (size 1.27 1.27)) hide)
-    )
-    (pin "1")
-    (pin "2")
-    (pin "3")
-    (pin "4")
-  )
   (symbol (lib_id "power:GND2") (at 172.212 122.428 0) (unit 1)
     (in_bom yes) (on_board yes)
@@
     )
     (pin "1")
+  )
+  (symbol (lib_id "Mechanical:MountingHole") (at 226.822 66.294 0) (unit 1)
+    (in_bom yes) (on_board yes) (fields_autoplaced)
+    (property "Reference" "H3" (id 0) (at 229.87 65.0239 0)
+      (effects (font (size 1.27 1.27)) (justify left))
+    )
+    (property "Value" "MountingHole" (id 1) (at 229.87 67.5639 0)
+      (effects (font (size 1.27 1.27)) (justify left))
+    )
+    (property "Footprint" "MountingHole:MountingHole_3.2mm_M3" (id 2) (at 226.822 66.294 0)
+      (effects (font (size 1.27 1.27)) hide)
+    )
+    (property "Datasheet" "~" (id 3) (at 226.822 66.294 0)
+      (effects (font (size 1.27 1.27)) hide)
+    )
   )
   (symbol (lib_id "power:+5VD") (at 76.454 122.428 0) (unit 1)
@@
     (pin "2")
   )
+  (symbol (lib_id "Mechanical:MountingHole") (at 226.822 56.134 0) (unit 1)
+    (in_bom yes) (on_board yes) (fields_autoplaced)
+    (property "Reference" "H1" (id 0) (at 229.87 54.8639 0)
+      (effects (font (size 1.27 1.27)) (justify left))
+    )
+    (property "Value" "MountingHole" (id 1) (at 229.87 57.4039 0)
+      (effects (font (size 1.27 1.27)) (justify left))
+    )
+    (property "Footprint" "MountingHole:MountingHole_3.2mm_M3" (id 2) (at 226.822 56.134 0)
+      (effects (font (size 1.27 1.27)) hide)
+    )
+    (property "Datasheet" "~" (id 3) (at 226.822 56.134 0)
+      (effects (font (size 1.27 1.27)) hide)
+    )
+  )
   (symbol (lib_id "Converter_DCDC:TEC2-1213WI") (at 96.012 49.022 0) (unit 1)
     (in_bom yes) (on_board yes) (fields_autoplaced)
@@
       (reference "D8") (unit 1) (value "LED_Small") (footprint "LED_SMD:LED_0805_2012Metric_Pad1.15x1.40mm_HandSolder")
     )
+    (path "/d77abb4e-9728-498d-9f77-c50ed71d858d"
+      (reference "H1") (unit 1) (value "MountingHole") (footprint "MountingHole:MountingHole_3.2mm_M3")
+    )
+    (path "/a826d4f1-aa41-4d34-8070-125b5f8ee214"
+      (reference "H3") (unit 1) (value "MountingHole") (footprint "MountingHole:MountingHole_3.2mm_M3")
+    )
     (path "/d0714426-20f0-4b37-aae0-9b121e6c9310"
       (reference "J1") (unit 1) (value "Conn_02x07_Odd_Even") (footprint "Connector_IDC:IDC-Header_2x07-1MP_P2.54mm_Latch_Vertical")
     )
-    (path "/1ebf09bd-2d15-4396-857b-c0ccf3cebbc9"
-      (reference "J2") (unit 1) (value "IGBT") (footprint "IGBT_Modul:IGBT_Gate")
-    )
     (path "/7640771e-5b32-4b09-8ee1-321e423562a0"
